File: ESPProgV1/ESPProgV1.kicad_pcb (KiCad board)
At the start: 2 copper layers, 22.4 x 46.6 mm, 21 parts, among them J1 USB_B_Micro, J2 Power, J3 header, Q1 S8050, Q2 S8050, U1 CH340G, Y1 Crystal

Commit message: BluePill board
BluePill board with STM32 microcontroller
Routing:
- added copper zone on B.Cu, net GND
- added copper zone on F.Cu, net GND
Changed lines of the file:
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@@
   (via (at 95.5 95.7) (size 0.8) (drill 0.4) (layers F.Cu B.Cu) (net 20))
   (segment (start 95.1 96.1) (end 95.5 95.7) (width 0.25) (layer F.Cu) (net 20))
+  (zone (net 1) (net_name GND) (layer F.Cu) (hatch edge 0.508)
+    (connect_pads (clearance 0.508))
+    (min_thickness 0.254)
+    (fill yes (arc_segments 32) (thermal_gap 0.508) (thermal_bridge_width 0.508))
+    (polygon
+      (pts
+        (xy 90.2 64.4) (xy 90.7 63.5) (xy 110.9 63.4) (xy 111.6 64.3) (xy 111.8 109.4)
+        (xy 111.6 109.7) (xy 90.1 109.7) (xy 89.7 109.4) (xy 89.7 63.5) (xy 90.7 63.5)
+      )
+    )
+  )
+  (zone (net 1) (net_name GND) (layer B.Cu) (hatch edge 0.508)
+    (connect_pads (clearance 0.508))
+    (min_thickness 0.254)
+    (fill yes (arc_segments 32) (thermal_gap 0.508) (thermal_bridge_width 0.508))
+    (polygon
+      (pts
+        (xy 111.9 63.4) (xy 111.9 109.5) (xy 111.8 109.7) (xy 90.1 109.7) (xy 89.7 109.4)
+        (xy 89.7 63.8) (xy 90 63.4) (xy 111.7 63.3)
+      )
+    )
+  )
 )
